File: testProject/testProject.kicad_sch (KiCad schematic)
At the start: 0 parts

Commit message: saving before I mess up
Parts:
- added C1: ~, symbol Device:C
- added R1, R2: ~, symbol Device:R
- added R3: R, symbol Device:R

Commit message: WIRE CONNECTION WORKS (not with exact pins)
Parts:
- removed C1: ~, symbol Device:C
- removed R1, R2: ~, symbol Device:R
- removed R3: R, symbol Device:R

Commit message: All good need to fix pin in kicad utils
Parts:
- added C1: (no value), symbol Device:C
- added D1: ED, symbol Device:LED
Connections:
- new net: C1.2, D1.1 (K)
- new net: C1.1, D1.2 (A)
Changed lines of the file:
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@@
 	(generator_version "8.0")
 	(paper "A4")
+ (wire
+		(pts
+			(xy 125.73 53.34) (xy 296.19 40)
+		)
+		(stroke
+			(width 0)
+			(type default)
+		)
+	)
+ (wire
+		(pts
+			(xy 118.11 53.34) (xy 303.81 40)
+		)
+		(stroke
+			(width 0)
+			(type default)
+		)
+	)
+ 	(symbol
+		(lib_id "Device:LED")
+		(at 121.92 53.34 0)
+		(unit 1)
+		(exclude_from_sim no)
+		(in_bom yes)
+		(on_board yes)
+		(dnp no)
+		(fields_autoplaced yes)
+		(property "Reference" "D1"
+			(at 121.92 53.34 0)
+			(effects
+				(font
+					(size 1.27 1.27)
+				)
+			)
+		)
+		(property "Value" "ED"
+			(at 121.92 53.34 0)
+			(effects
+				(font
+					(size 1.27 1.27)
+				)
+			)
+		)
+		(property "Footprint" ""
+			(at 121.92 53.34 0)
+			(effects
+				(font
+					(size 1.27 1.27)
+				)
+				(hide yes)
+			)
+		)
+		(property "Datasheet" "~"
+			(at 121.92 53.34 0)
+			(effects
+				(font
+					(size 1.27 1.27)
+				)
+				(hide yes)
+			)
+		)
+		(property "Description" "ight emitting diode"
+			(at 121.92 53.34 0)
+			(effects
+				(font
+					(size 1.27 1.27)
+				)
+				(hide yes)
+			)
+		)
+		(pin "1"
+		)
+		(pin "2"
+		)
+		(instances
+			(project "testProject"
+				(path "/dea647a7-e0d8-45e4-9bce-23c7e387cf2b"
+					(reference "D1")
+					(unit 1)
+				)
+			)
+		)
+	)
+	(symbol
+		(lib_id "Device:C")
+		(at 300 40 90)
+		(unit 1)
+		(exclude_from_sim no)
+		(in_bom yes)
+		(on_board yes)
+		(dnp no)
+		(fields_autoplaced yes)
+		(property "Reference" "C1"
+			(at 300 40 0)
+			(effects
+				(font
+					(size 1.27 1.27)
+				)
+			)
+		)
+		(property "Value" ""
+			(at 300 40 0)
+			(effects
+				(font
+					(size 1.27 1.27)
+				)
+			)
+		)
+		(property "Footprint" ""
+			(at 300 40 0)
+			(effects
+				(font
+					(size 1.27 1.27)
+				)
+				(hide yes)
+			)
+		)
+		(property "Datasheet" "~"
+			(at 300 40 0)
+			(effects
+				(font
+					(size 1.27 1.27)
+				)
+				(hide yes)
+			)
+		)
+		(property "Description" "npolarized capacitor"
+			(at 300 40 0)
+			(effects
+				(font
+					(size 1.27 1.27)
+				)
+				(hide yes)
+			)
+		)
+		(pin "1"
+		)
+		(pin "2"
+		)
+		(instances
+			(project "testProject"
+				(path "/dea647a7-e0d8-45e4-9bce-23c7e387cf2b"
+					(reference "C1")
+					(unit 1)
+				)
+			)
+		)
+	)
 	(sheet_instances
 		(path "/"

Commit message: integrated GUI
Parts:
- removed C1: (no value), symbol Device:C
- removed D1: ED, symbol Device:LED
Changed lines of the file:
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@@
 	(generator_version "8.0")
 	(paper "A4")
- (wire
-		(pts
-			(xy 125.73 53.34) (xy 296.19 40)
-		)
-		(stroke
-			(width 0)
-			(type default)
-		)
-	)
- (wire
-		(pts
-			(xy 118.11 53.34) (xy 303.81 40)
-		)
-		(stroke
-			(width 0)
-			(type default)
-		)
-	)
- 	(symbol
-		(lib_id "Device:LED")
-		(at 121.92 53.34 0)
-		(unit 1)
-		(exclude_from_sim no)
-		(in_bom yes)
-		(on_board yes)
-		(dnp no)
-		(fields_autoplaced yes)
-		(property "Reference" "D1"
-			(at 121.92 53.34 0)
-			(effects
-				(font
-					(size 1.27 1.27)
-				)
-			)
-		)
-		(property "Value" "ED"
-			(at 121.92 53.34 0)
-			(effects
-				(font
-					(size 1.27 1.27)
-				)
-			)
-		)
-		(property "Footprint" ""
-			(at 121.92 53.34 0)
-			(effects
-				(font
-					(size 1.27 1.27)
-				)
-				(hide yes)
-			)
-		)
-		(property "Datasheet" "~"
-			(at 121.92 53.34 0)
-			(effects
-				(font
-					(size 1.27 1.27)
-				)
-				(hide yes)
-			)
-		)
-		(property "Description" "ight emitting diode"
-			(at 121.92 53.34 0)
-			(effects
-				(font
-					(size 1.27 1.27)
-				)
-				(hide yes)
-			)
-		)
-		(pin "1"
-		)
-		(pin "2"
-		)
-		(instances
-			(project "testProject"
-				(path "/dea647a7-e0d8-45e4-9bce-23c7e387cf2b"
-					(reference "D1")
-					(unit 1)
-				)
-			)
-		)
-	)
-	(symbol
-		(lib_id "Device:C")
-		(at 300 40 90)
-		(unit 1)
-		(exclude_from_sim no)
-		(in_bom yes)
-		(on_board yes)
-		(dnp no)
-		(fields_autoplaced yes)
-		(property "Reference" "C1"
-			(at 300 40 0)
-			(effects
-				(font
-					(size 1.27 1.27)
-				)
-			)
-		)
-		(property "Value" ""
-			(at 300 40 0)
-			(effects
-				(font
-					(size 1.27 1.27)
-				)
-			)
-		)
-		(property "Footprint" ""
-			(at 300 40 0)
-			(effects
-				(font
-					(size 1.27 1.27)
-				)
-				(hide yes)
-			)
-		)
-		(property "Datasheet" "~"
-			(at 300 40 0)
-			(effects
-				(font
-					(size 1.27 1.27)
-				)
-				(hide yes)
-			)
-		)
-		(property "Description" "npolarized capacitor"
-			(at 300 40 0)
-			(effects
-				(font
-					(size 1.27 1.27)
-				)
-				(hide yes)
-			)
-		)
-		(pin "1"
-		)
-		(pin "2"
-		)
-		(instances
-			(project "testProject"
-				(path "/dea647a7-e0d8-45e4-9bce-23c7e387cf2b"
-					(reference "C1")
-					(unit 1)
-				)
-			)
-		)
-	)
 	(sheet_instances
 		(path "/"
